File: hw/main_fpga.sch (KiCad schematic (older format))
At the start: 45 parts

Commit message: Adding plugfects submodules
Adding
- plugfects/plugmodules - kicad ciruit modules
- plugfects/pluglib - kicad component libraries
- Fix path to use the new location
Parts:
- C16, C17, C18, C19, C20, C21, C24, C27, C28, C29, C31, C33, C34, C35, C37, C39, C40, C41, C43, C45, C46, C47, C49, C50, C51: renamed from C?; footprint (none) -> Capacitors_SMD:C_0603_HandSoldering
- U4: renamed from U?; footprint (none) -> Housings_QFP:TQFP-144_20x20mm_Pitch0.5mm
- gave numbers to parts that had none: 16
